Commit message: Added table avoidance simulation. Currently only takes in to account Z direction repulsion forces.

File: elfin/elfin_description/urdf/box.urdf.xacro (robot description, xacro)
@@ -25,13 +25,13 @@
     <static> true </static>
     <visual>
-      <origin xyz="0.5 0 0.05" rpy="0 0 0" />
+      <origin xyz="-0.55 0 0.3" rpy="0 0 0" />
       <geometry>
-         <box size="0.7 0.5 0.1"/>
+         <box size="0.7 0.5 0.04"/>
       </geometry>
     </visual>
     <collision>
-      <origin xyz="0.5 0 0.05" rpy="0 0 0" />
+      <origin xyz="-0.55 0 0.3" rpy="0 0 0" />
       <geometry>
-         <box size="0.7 0.5 0.1"/>
+         <box size="0.7 0.5 0.04"/>
       </geometry>
     </collision>
